File: RP2354B_core.kicad_block/RP2354B_core.kicad_sch (KiCad schematic)
At the start: 22 parts, among them U1 RP2350_80QFN, Y1 ABM8-272-T3

Commit message: Renumber block components sequentially (C1..C17, R1..R2)
Closes refdes gaps that caused duplicate footprints when importing the
block PCB into parent projects via re-link by refdes.
Parts:
- renumbered C3 to C1, C13 to C10, C14 to C11, C15 to C12, C16 to C13, C17 to C14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
Other:
- moved on the sheet: C1, C2, R1, Y1
